File: Hardware/TR v0.1.sch (KiCad schematic (older format))
At the start: 50 parts, among them IC1 ATmega328PB-AU, J1 Input, J2 OutputAll, J3 Delay CV1, J4 Delay CV2, J5 Delay CV3, J6 OutputOne, J7 OutputTwo, J8 OutputThree, Q1 BC847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

Commit message: Added Trigger Outputs
Parts:
- added R11, R20, R6, R7: 1K, Resistor_SMD:R_0603_1608Metric, symbol Device:R
Connections:
- net D2: now also R6.1; no longer J2.3
- net D4: now also R7.1; no longer J6.3
- net D7: now also R11.1; no longer J7.3
- net D8: now also R20.1; no longer J8.3
- new net: J2.3, R6.2
- new net: J6.3, R7.2
- new net: J7.3, R11.2
- new net: J8.3, R20.2
Changed lines of the file:
@@
 Wire Wire Line
 	10150 1950 10150 2050
-Text GLabel 10250 2250 2    50   Input ~ 0
+Text GLabel 10550 2250 2    50   Input ~ 0
 D2
 Wire Wire Line
@@
 	9600 2950 10150 2950
 Connection ~ 10150 2950
-Text GLabel 10250 2750 2    50   Input ~ 0
+Text GLabel 10550 2750 2    50   Input ~ 0
 D4
 Wire Wire Line
@@
 Wire Wire Line
 	10150 3950 10150 4100
-Text GLabel 10250 3250 2    50   Input ~ 0
+Text GLabel 10550 3250 2    50   Input ~ 0
 D7
 Wire Wire Line
@@
 	0    1    1    0
 $EndComp
-Text GLabel 10250 3750 2    50   Input ~ 0
+Text GLabel 10550 3750 2    50   Input ~ 0
 D8
 $Comp
@@
 	1    0    0    -1
 $EndComp
+$Comp
+L Device:R R6
+U 1 1 606B9DBE
+P 10400 2250
+F 0 "R6" V 10300 2150 50  0000 C CNN
+F 1 "1K" V 10300 2300 50  0000 C CNN
+F 2 "Resistor_SMD:R_0603_1608Metric" V 10330 2250 50  0001 C CNN
+F 3 "~" H 10400 2250 50  0001 C CNN
+	1    10400 2250
+	0    1    1    0
+$EndComp
+$Comp
+L Device:R R7
+U 1 1 606BA97F
+P 10400 2750
+F 0 "R7" V 10300 2650 50  0000 C CNN
+F 1 "1K" V 10300 2800 50  0000 C CNN
+F 2 "Resistor_SMD:R_0603_1608Metric" V 10330 2750 50  0001 C CNN
+F 3 "~" H 10400 2750 50  0001 C CNN
+	1    10400 2750
+	0    1    1    0
+$EndComp
+$Comp
+L Device:R R11
+U 1 1 606BB499
+P 10400 3250
+F 0 "R11" V 10300 3150 50  0000 C CNN
+F 1 "1K" V 10300 3300 50  0000 C CNN
+F 2 "Resistor_SMD:R_0603_1608Metric" V 10330 3250 50  0001 C CNN
+F 3 "~" H 10400 3250 50  0001 C CNN
+	1    10400 3250
+	0    1    1    0
+$EndComp
+$Comp
+L Device:R R20
+U 1 1 606BB80B
+P 10400 3750
+F 0 "R20" V 10300 3650 50  0000 C CNN
+F 1 "1K" V 10300 3800 50  0000 C CNN
+F 2 "Resistor_SMD:R_0603_1608Metric" V 10330 3750 50  0001 C CNN
+F 3 "~" H 10400 3750 50  0001 C CNN
+	1    10400 3750
+	0    1    1    0
+$EndComp
 $EndSCHEMATC
